Commit message: Simulation update

File: mechanics/urdf/UR5_simplified/urdf/UR5_simplified.urdf (robot description, URDF)
Before this commit: robot UR5_simplified, 8 links, 7 joints
Joints:
- joint j1: limit lower=-4.7124 upper=0 effort=0 velocity=0 -> lower=-4.7124 upper=0 effort=150 velocity=150
- joint j2: limit lower=0 upper=1.5708 effort=0 velocity=0 -> lower=0 upper=1.5708 effort=150 velocity=150
- joint j3: limit lower=-2.0944 upper=2.0944 effort=0 velocity=0 -> lower=-2.0944 upper=2.0944 effort=150 velocity=150
- joint j4: limit lower=-3.1416 upper=0 effort=0 velocity=0 -> lower=-3.1416 upper=0 effort=150 velocity=150
- joint j5: limit lower=-4.7124 upper=0 effort=0 velocity=0 -> lower=-4.7124 upper=0 effort=150 velocity=150
- joint j6: limit lower=-4.7124 upper=0 effort=0 velocity=0 -> lower=-4.7124 upper=0 effort=150 velocity=150
